File: kicad/carrier_board/carrier_board.kicad_sch (KiCad schematic)
At the start: 3 parts

Commit message: schematic progress
Parts:
- added BuckConverter: Conn_01x02, Connector_PinSocket_2.54mm:PinSocket_1x03_P2.54mm_Vertical, symbol Connector_Generic:Conn_01x02
- added C1: 22µf, symbol Device:C
- added C2, C4, C5: 100nf, symbol Device:C
- added C3: 10µf, symbol Device:C
- added D1, D2, D3: LED, LED_THT:LED_D5.0mm, symbol Device:LED
- added PiUSB, RecordingButton: Conn_01x02, Connector_PinHeader_2.54mm:PinHeader_1x02_P2.54mm_Vertical, symbol Connector_Generic:Conn_01x02
- added R1, R2, R3: R, Resistor_THT:R_Axial_DIN0207_L6.3mm_D2.5mm_P10.16mm_Horizontal, symbol Device:R
- added R4: 4k7, Resistor_THT:R_Axial_DIN0207_L6.3mm_D2.5mm_P10.16mm_Horizontal, symbol Device:R
- added R5: 330, Resistor_THT:R_Axial_DIN0207_L6.3mm_D2.5mm_P10.16mm_Horizontal, symbol Device:R
Connections:
- net GND: now reaches SPIMicroSDBreakout.1 (GND)
- net GND: now also A1.13 (GND), A1.18 (GND), A1.23 (GND), A1.28 (GND), A1.3 (GND), A1.33 (AGND), A1.38 (GND), A1.8 (GND), USBCBreakoutBoard.8 (GND), BuckConverter.2 (-), C1.2, C2.2, C3.2, C4.2, C5.2, R1.1, R2.1, R3.1, RecordingButton.2 (Pin_2)
- net MISO: now reaches SPIMicroSDBreakout.2 (MISO)
- net MISO: now also A1.16 (GPIO12)
- net SCK: now reaches SPIMicroSDBreakout.3 (CLK)
- net SCK: now also A1.14 (GPIO10)
- net MOSI: now reaches SPIMicroSDBreakout.4 (MOSI)
- net MOSI: now also A1.15 (GPIO11)
- net CS: now reaches SPIMicroSDBreakout.5 (CS)
- net CS: now also A1.17 (GPIO13)
- net +3.3V: now reaches SPIMicroSDBreakout.6 (3v3)
- net +3.3V: now also A1.36 (3V3), D1.2 (A)
- net D+: now reaches USBCBreakoutBoard.3 (D+)
- net D+: now also PiUSB.1 (D+)
- net D-: now reaches USBCBreakoutBoard.4 (D-)
- net D-: now also PiUSB.2 (D-)
- net USB5v: now reaches USBCBreakoutBoard.7 (VBUS)
- net USB5v: now also A1.40 (VBUS)
- net LED_USB: now reaches A1.11 (GPIO8)
- net LED_USB: now also D3.2 (A)
- net +5V: now reaches A1.39 (VSYS)
- net +5V: now also BuckConverter.1 (+), C1.1, C2.1
- net BTN_REC: now reaches A1.4 (GPIO2)
- net BTN_REC: now also R5.1
- net LED_REC: now reaches A1.5 (GPIO3)
- net LED_REC: now also D2.2 (A)
- new net: C5.1, R4.2, R5.2, RecordingButton.1 (Pin_1)
- new net: D2.1 (K), R2.2
- new net: D3.1 (K), R3.2
- new net: D1.1 (K), R1.2
- new net +3V3: C3.1, C4.1, R4.1
Other:
- note added: "Deutsch Connector"
- note added: "LED Circuit"
- note added: "RaspberryPi Pico W SD DAQ"
- note added: "Raspberrypi Pico W"
- note added: "SD Breakout"
- note added: "Supply Decoupling"
- note added: "USB C Breakout"
- moved on the sheet: A1, SPIMicroSDBreakout, USBCBreakoutBoard
